Commit message: fixed description and format of gazebo.launch.py

File: src/gazebo/description/robot.urdf.xacro (robot description, xacro)
@@ -1,41 +1,63 @@
 <?xml version="1.0"?>
-<robot xmlns:xacro="http://www.ros.org/wiki/xacro" name="stock_car">
+<robot xmlns:xacro="http://www.ros.org/wiki/xacro" name="four_wheel_robot">
+  <!-- Dimensions are in metres. The chassis mass is a temporary placeholder. -->
+  <xacro:property name="chassis_mass" value="1.0"/>
+  <xacro:property name="wheel_radius" value="0.035"/>
+  <xacro:property name="driven_wheel_width" value="0.026"/>
+  <xacro:property name="omni_wheel_width" value="0.012"/>
+  <xacro:property name="wheel_separation" value="0.161"/>
+  <xacro:property name="wheel_x" value="-0.026"/>
+  <xacro:property name="wheel_z" value="${wheel_radius}"/>
+  <xacro:property name="omni_x" value="0.031"/>
+  <xacro:property name="omni_y" value="0.007"/>
+  <xacro:property name="chassis_bottom" value="0.011"/>
+  <xacro:property name="chassis_height" value="0.048"/>
+  <material name="red">
+    <color rgba="0.8 0.0 0.0 1.0"/>
+  </material>
+  <material name="black">
+    <color rgba="0.05 0.05 0.05 1.0"/>
+  </material>
   <link name="base_link">
+    <inertial>
+      <origin xyz="0 0 0"/>
+      <mass value="${chassis_mass}"/>
+      <inertia ixx="0.01" ixy="0.0" ixz="0.0"
+               iyy="0.01" iyz="0.0" izz="0.01"/>
+    </inertial>
     <visual>
-      <origin xyz="0 0 0.4"/>
+      <origin xyz="0 0 ${chassis_bottom}"/>
       <geometry>
-        <box size="2.0 1.0 0.5"/>
+        <mesh filename="package://gazebo/description/chassis.stl"
+              scale="1 1 4.8"/>
       </geometry>
-      <material name="blue">
-        <color rgba="0 0 1 1"/>
-      </material>
+      <material name="red"/>
     </visual>
     <collision>
-      <origin xyz="0 0 0.4"/>
+      <origin xyz="0 0 ${chassis_bottom}"/>
       <geometry>
-        <box size="2.0 1.0 0.5"/>
+        <mesh filename="package://gazebo/description/chassis.stl"
+              scale="1 1 4.8"/>
       </geometry>
     </collision>
-    <inertial>
-      <origin xyz="0 0 0.4"/>
-      <mass value="1.14395"/>
-      <inertia ixx="0.095329" ixy="0" ixz="0" iyy="0.381317" iyz="0" izz="0.476646"/>
-    </inertial>
   </link>
-  <xacro:macro name="wheel" params="name y">
+  <xacro:macro name="driven_wheel" params="name y">
     <link name="${name}">
+      <inertial>
+        <mass value="0.2"/>
+        <inertia ixx="0.0002" ixy="0.0" ixz="0.0"
+                 iyy="0.0001" iyz="0.0" izz="0.0002"/>
+      </inertial>
       <visual>
-        <origin rpy="-1.5708 0 0"/>
+        <origin rpy="${pi / 2} 0 0"/>
         <geometry>
-          <cylinder radius="0.4" length="0.2"/>
+          <cylinder radius="${wheel_radius}" length="${driven_wheel_width}"/>
         </geometry>
-        <material name="red">
-          <color rgba="1 0 0 1"/>
-        </material>
+        <material name="black"/>
       </visual>
       <collision>
-        <origin rpy="-1.5708 0 0"/>
+        <origin rpy="${pi / 2} 0 0"/>
         <geometry>
-          <cylinder radius="0.4" length="0.2"/>
+          <cylinder radius="${wheel_radius}" length="${driven_wheel_width}"/>
         </geometry>
       </collision>
@@ -44,29 +66,68 @@
       <parent link="base_link"/>
       <child link="${name}"/>
-      <origin xyz="-0.5 ${y} 0"/>
+      <origin xyz="${wheel_x} ${y} ${wheel_z}"/>
       <axis xyz="0 1 0"/>
     </joint>
+    <gazebo reference="${name}">
+      <mu1>1.0</mu1>
+      <mu2>1.0</mu2>
+    </gazebo>
   </xacro:macro>
-  <xacro:wheel name="left_wheel" y="0.6"/>
-  <xacro:wheel name="right_wheel" y="-0.6"/>
-  <link name="caster">
-    <visual>
-      <geometry>
-        <sphere radius="0.2"/>
-      </geometry>
-      <material name="green">
-        <color rgba="0 1 0 1"/>
-      </material>
-    </visual>
-    <collision>
-      <geometry>
-        <sphere radius="0.2"/>
-      </geometry>
-    </collision>
-  </link>
-  <joint name="caster_joint" type="fixed">
-    <parent link="base_link"/>
-    <child link="caster"/>
-    <origin xyz="0.8 0 -0.2"/>
-  </joint>
+  <xacro:macro name="omni_wheel" params="name y">
+    <link name="${name}">
+      <inertial>
+        <mass value="0.1"/>
+        <inertia ixx="0.0001" ixy="0.0" ixz="0.0"
+                 iyy="0.00005" iyz="0.0" izz="0.0001"/>
+      </inertial>
+      <visual>
+        <origin rpy="${pi / 2} 0 0"/>
+        <geometry>
+          <cylinder radius="${wheel_radius}" length="${omni_wheel_width}"/>
+        </geometry>
+        <material name="black"/>
+      </visual>
+      <collision>
+        <origin rpy="${pi / 2} 0 0"/>
+        <geometry>
+          <cylinder radius="${wheel_radius}" length="${omni_wheel_width}"/>
+        </geometry>
+      </collision>
+    </link>
+    <joint name="${name}_joint" type="continuous">
+      <parent link="base_link"/>
+      <child link="${name}"/>
+      <origin xyz="${omni_x} ${y} ${wheel_z}"/>
+      <axis xyz="0 1 0"/>
+    </joint>
+    <gazebo reference="${name}">
+      <mu1>0.01</mu1>
+      <mu2>0.01</mu2>
+    </gazebo>
+  </xacro:macro>
+  <xacro:driven_wheel name="left_wheel" y="${wheel_separation / 2}"/>
+  <xacro:driven_wheel name="right_wheel" y="${-wheel_separation / 2}"/>
+  <xacro:omni_wheel name="front_omni_left" y="${omni_y}"/>
+  <xacro:omni_wheel name="front_omni_right" y="${-omni_y}"/>
+  <gazebo>
+    <plugin
+      filename="libignition-gazebo-diff-drive-system.so"
+      name="ignition::gazebo::systems::DiffDrive">
+      <left_joint>left_wheel_joint</left_joint>
+      <right_joint>right_wheel_joint</right_joint>
+      <wheel_separation>${wheel_separation}</wheel_separation>
+      <wheel_radius>${wheel_radius}</wheel_radius>
+      <odom_publish_frequency>50</odom_publish_frequency>
+      <topic>/cmd_vel</topic>
+      <odom_topic>/odom</odom_topic>
+      <tf_topic>/tf</tf_topic>
+      <frame_id>odom</frame_id>
+      <child_frame_id>base_link</child_frame_id>
+    </plugin>
+    <plugin
+      filename="libignition-gazebo-joint-state-publisher-system.so"
+      name="ignition::gazebo::systems::JointStatePublisher">
+      <topic>/model/four_wheel_robot/joint_state</topic>
+    </plugin>
+  </gazebo>
 </robot>
